Commit message: Close the lab-arm twin's gripper on the pen (#39)
The twin froze the xArm Gripper's six finger joints at their zero pose,
which is fully open (~85 mm), so the pen hung between open fingers. The
URDF builder can now freeze joints at a drive angle, baking each mimic
joint's rotation into its fixed origin; generate_xarm7_urdf.py --real uses
--gripper-closure-rad 0.76 (pads ~9.9 mm apart on the 10 mm pen) until the
lab arm's reading replaces it. xarm7_real.urdf changes only those six
origins; xarm7_real.usd was re-imported from it (meshes still embedded).
Drawing is unaffected: ACT on Cat 1163bceaf6134cf5 in the twin, 0.257 mm.

Also moves the video close-up camera low and to the side (top-down, the
wrist hid the sheet) and clears old videos before assembling new ones.

File: isaac-sim/assets/xarm7/xarm7_real.urdf (robot description, URDF)
Before this commit: robot xarm7_real, 20 links, 19 joints
Joints:
- joint drive_joint: origin xyz=0 0.035 0.059098 rpy=0 0 0 -> xyz=0 0.035 0.059098 rpy=0.76 -0 0
- joint left_finger_joint: origin xyz=0 0.035465 0.042039 rpy=0 0 0 -> xyz=0 0.035465 0.042039 rpy=-0.76 -0 0
- joint left_inner_knuckle_joint: origin xyz=0 0.02 0.074098 rpy=0 0 0 -> xyz=0 0.02 0.074098 rpy=0.76 -0 0
- joint right_finger_joint: origin xyz=0 -0.035465 0.042039 rpy=0 0 0 -> xyz=0 -0.035465 0.042039 rpy=0.76 -0 0
- joint right_inner_knuckle_joint: origin xyz=0 -0.02 0.074098 rpy=0 0 0 -> xyz=0 -0.02 0.074098 rpy=-0.76 -0 0
- joint right_outer_knuckle_joint: origin xyz=0 -0.035 0.059098 rpy=0 0 0 -> xyz=0 -0.035 0.059098 rpy=-0.76 -0 0
